File: Hardware/RPU-8_PC_8/RPU-8_PC_8.kicad_sch (KiCad schematic)
At the start: 8 parts, among them J1 ADDR_BUS, J2 DATA_BUS, J3 Conn_01x03_Female, J4 CTRL_BUS, J5 INST_REG, U1 74HC161, U2 74HC245, U3 74HC161

Commit message: updated TODO.md
Parts:
- added C1, C2, C3: 0.1 uF, symbol Device:C
Connections:
- net +5V: now also C1.1, C2.1, C3.1
- net GND: now also C1.2, C2.2, C3.2
Changed lines of the file:
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@@
 (kicad_sch (version 20211123) (generator eeschema)
   (paper "A4")
+  (junction (at 68.58 68.58) (diameter 0) (color 0 0 0 0)
+  )
+  (junction (at 68.58 76.2) (diameter 0) (color 0 0 0 0)
+  )
   (junction (at 172.72 55.88) (diameter 0) (color 0 0 0 0)
   )
+  (junction (at 76.2 76.2) (diameter 0) (color 0 0 0 0)
+  )
+  (junction (at 76.2 68.58) (diameter 0) (color 0 0 0 0)
+  )
   (junction (at 175.26 55.88) (diameter 0) (color 0 0 0 0)
   )
@@
   (junction (at 31.75 99.06) (diameter 0) (color 0 0 0 0)
   )
+  (wire (pts (xy 57.15 76.2) (xy 68.58 76.2))
+    (stroke (width 0) (type default) (color 0 0 0 0))
+  )
+  (wire (pts (xy 68.58 68.58) (xy 76.2 68.58))
+    (stroke (width 0) (type default) (color 0 0 0 0))
+  )
+  (wire (pts (xy 76.2 76.2) (xy 83.82 76.2))
+    (stroke (width 0) (type default) (color 0 0 0 0))
+  )
   (wire (pts (xy 138.43 88.9) (xy 138.43 113.03))
     (stroke (width 0) (type default) (color 0 0 0 0))
@@
     (stroke (width 0) (type default) (color 0 0 0 0))
   )
+  (wire (pts (xy 68.58 76.2) (xy 76.2 76.2))
+    (stroke (width 0) (type default) (color 0 0 0 0))
+  )
   (wire (pts (xy 125.73 53.34) (xy 125.73 63.5))
     (stroke (width 0) (type default) (color 0 0 0 0))
   )
+  (wire (pts (xy 76.2 68.58) (xy 83.82 68.58))
+    (stroke (width 0) (type default) (color 0 0 0 0))
+  )
   (wire (pts (xy 172.72 55.88) (xy 172.72 63.5))
     (stroke (width 0) (type default) (color 0 0 0 0))
@@
   )
   (wire (pts (xy 143.51 88.9) (xy 143.51 113.03))
+    (stroke (width 0) (type default) (color 0 0 0 0))
+  )
+  (wire (pts (xy 57.15 68.58) (xy 68.58 68.58))
     (stroke (width 0) (type default) (color 0 0 0 0))
   )
@@
     (pin "9")
   )
+  (symbol (lib_id "power:+5V") (at 57.15 68.58 180) (unit 1)
+    (in_bom yes) (on_board yes) (fields_autoplaced)
+    (property "Reference" "#PWR03" (id 0) (at 57.15 64.77 0)
+      (effects (font (size 1.27 1.27)) hide)
+    )
+    (property "Value" "+5V" (id 1) (at 59.69 69.8499 0)
+      (effects (font (size 1.27 1.27)) (justify right))
+    )
+    (property "Footprint" "" (id 2) (at 57.15 68.58 0)
+      (effects (font (size 1.27 1.27)) hide)
+    )
+    (property "Datasheet" "" (id 3) (at 57.15 68.58 0)
+      (effects (font (size 1.27 1.27)) hide)
+    )
+    (pin "1")
+  )
   (symbol (lib_id "power:GND") (at 110.49 76.2 0) (unit 1)
     (in_bom yes) (on_board yes) (fields_autoplaced)
@@
     (pin "1")
   )
+  (symbol (lib_id "power:GND") (at 57.15 76.2 0) (unit 1)
+    (in_bom yes) (on_board yes)
+    (property "Reference" "#PWR013" (id 0) (at 57.15 82.55 0)
+      (effects (font (size 1.27 1.27)) hide)
+    )
+    (property "Value" "GND" (id 1) (at 57.15 81.28 0))
+    (property "Footprint" "" (id 2) (at 57.15 76.2 0)
+      (effects (font (size 1.27 1.27)) hide)
+    )
+    (property "Datasheet" "" (id 3) (at 57.15 76.2 0)
+      (effects (font (size 1.27 1.27)) hide)
+    )
+    (pin "1")
+  )
+  (symbol (lib_id "Device:C") (at 83.82 72.39 0) (unit 1)
+    (in_bom yes) (on_board yes) (fields_autoplaced)
+    (property "Reference" "C3" (id 0) (at 87.63 71.1199 0)
+      (effects (font (size 1.27 1.27)) (justify left))
+    )
+    (property "Value" "0.1 uF" (id 1) (at 87.63 73.6599 0)
+      (effects (font (size 1.27 1.27)) (justify left))
+    )
+    (property "Footprint" "" (id 2) (at 84.7852 76.2 0)
+      (effects (font (size 1.27 1.27)) hide)
+    )
+    (property "Datasheet" "~" (id 3) (at 83.82 72.39 0)
+      (effects (font (size 1.27 1.27)) hide)
+    )
+    (pin "1")
+    (pin "2")
+  )
   (symbol (lib_id "Connector:Conn_01x08_Female") (at 22.86 168.91 180) (unit 1)
     (in_bom yes) (on_board yes) (fields_autoplaced)
@@
     )
     (pin "1")
+  )
+  (symbol (lib_id "Device:C") (at 68.58 72.39 0) (unit 1)
+    (in_bom yes) (on_board yes) (fields_autoplaced)
+    (property "Reference" "C1" (id 0) (at 72.39 71.1199 0)
+      (effects (font (size 1.27 1.27)) (justify left))
+    )
+    (property "Value" "0.1 uF" (id 1) (at 72.39 73.6599 0)
+      (effects (font (size 1.27 1.27)) (justify left))
+    )
+    (property "Footprint" "" (id 2) (at 69.5452 76.2 0)
+      (effects (font (size 1.27 1.27)) hide)
+    )
+    (property "Datasheet" "~" (id 3) (at 68.58 72.39 0)
+      (effects (font (size 1.27 1.27)) hide)
+    )
+    (pin "1")
+    (pin "2")
   )
   (symbol (lib_id "74xx:74HC245") (at 148.59 125.73 90) (unit 1)
@@
     (pin "1")
   )
+  (symbol (lib_id "Device:C") (at 76.2 72.39 0) (unit 1)
+    (in_bom yes) (on_board yes) (fields_autoplaced)
+    (property "Reference" "C2" (id 0) (at 80.01 71.1199 0)
+      (effects (font (size 1.27 1.27)) (justify left))
+    )
+    (property "Value" "0.1 uF" (id 1) (at 80.01 73.6599 0)
+      (effects (font (size 1.27 1.27)) (justify left))
+    )
+    (property "Footprint" "" (id 2) (at 77.1652 76.2 0)
+      (effects (font (size 1.27 1.27)) hide)
+    )
+    (property "Datasheet" "~" (id 3) (at 76.2 72.39 0)
+      (effects (font (size 1.27 1.27)) hide)
+    )
+    (pin "1")
+    (pin "2")
+  )
   (symbol (lib_id "Connector:Conn_01x16_Female") (at 22.86 43.18 180) (unit 1)
     (in_bom yes) (on_board yes) (fields_autoplaced)
@@
     (pin "9")
   )
-  (symbol (lib_id "power:GND") (at 67.31 68.58 0) (unit 1)
-    (in_bom yes) (on_board yes) (fields_autoplaced)
-    (property "Reference" "#PWR03" (id 0) (at 67.31 74.93 0)
-      (effects (font (size 1.27 1.27)) hide)
-    )
-    (property "Value" "GND" (id 1) (at 67.31 73.66 0))
-    (property "Footprint" "" (id 2) (at 67.31 68.58 0)
-      (effects (font (size 1.27 1.27)) hide)
-    )
-    (property "Datasheet" "" (id 3) (at 67.31 68.58 0)
-      (effects (font (size 1.27 1.27)) hide)
-    )
-    (pin "1")
-  )
   (sheet_instances
     (path "/" (page "1"))
@@
       (reference "#PWR02") (unit 1) (value "GND") (footprint "")
     )
-    (path "/fc91997e-d1f8-40c9-b23e-76612ec71681"
-      (reference "#PWR03") (unit 1) (value "GND") (footprint "")
+    (path "/6014ad9f-c15f-4b0d-a5a5-bdc274037976"
+      (reference "#PWR03") (unit 1) (value "+5V") (footprint "")
     )
     (path "/6fe48ac3-d9b5-4921-8e7d-7df2d82ed285"
@@
       (reference "#PWR012") (unit 1) (value "+5V") (footprint "")
     )
+    (path "/96cb244d-961a-4218-8d99-242e90e72d26"
+      (reference "#PWR013") (unit 1) (value "GND") (footprint "")
+    )
+    (path "/d7e51fc8-b5ff-4106-bef0-2aa74c6173e8"
+      (reference "C1") (unit 1) (value "0.1 uF") (footprint "")
+    )
+    (path "/ed9379ae-e09a-4c92-bebb-88d86020ad75"
+      (reference "C2") (unit 1) (value "0.1 uF") (footprint "")
+    )
+    (path "/9c4096cc-0566-4abe-b24f-8f08537b79c1"
+      (reference "C3") (unit 1) (value "0.1 uF") (footprint "")
+    )
     (path "/f8bad4e8-5155-40b8-b53b-db6ad5f95837"
