File: Hardware/RPU-8_LEDS/RPU-8_LEDS.kicad_sch (KiCad schematic)
At the start: 17 parts, among them J1 ADDR_BUS, J2 DATA_BUS, J3 Conn_01x03_Female, J4 CTRL_BUS, J5 INST_REG, U1 8_Segment_LED_Bar_Graph, U2 8_Segment_LED_Bar_Graph, U3 8_Segment_LED_Bar_Graph, U4 8_Segment_LED_Bar_Graph, U5 8_Segment_LED_Bar_Graph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

Commit message: added images
Parts:
- added D1: LED, Connector_PinHeader_2.54mm:PinHeader_1x02_P2.54mm_Horizontal, symbol Device:LED
- added J6: Barrel_Jack, Connector_BarrelJack:BarrelJack_Horizontal, symbol Connector:Barrel_Jack
- added SW1: SW_Push, Button_Switch_THT:SW_PUSH_6mm, symbol Switch:SW_Push
- DATA_BUS: renamed from U1; value 8_Segment_LED_Bar_Graph -> DATA_BUS
- U4: value 8_Segment_LED_Bar_Graph -> INST
- renumbered U2 to ADDR_BUS, U6 to INST_ADDR
Connections:
- net +5V: now also J6.2, SW1.1
- net CLK: now also D1.2 (A)
- net GND: now also D1.1 (K), J6.1
- net RST: now also SW1.2
