File: Hardware/RPU-8_CTRL/RPU-8_CTRL.kicad_pcb (KiCad board)
At the start: 4 copper layers, 138.4 x 57.2 mm, 8 parts, among them J1 ADDR_BUS, J2 DATA_BUS, J3 Conn_01x03_Female, J4 CTRL_BUS, U1 AT28C16, U2 AT28C16, U3 AT28C16

Commit message: CTRL Board Layout Fixed
Parts:
- added J5: INST_REG, Connector_PinSocket_2.54mm:PinSocket_1x08_P2.54mm_Vertical, F.Cu at (127.0, 119.5)
- moved J2 40.5 mm to (128.3, 73.6), turned to -90 degrees
- moved J1 39.4 mm to (170.2, 73.6), turned to -90 degrees
- moved J3 10.1 mm to (94.0, 92.7)
Routing:
- net D2: track 10.7 -> 46.5 mm
- net D0: track 11.8 -> 45.4 mm
- net D3: track 10.7 -> 43.7 mm
- net D1: track 11.8 -> 42.1 mm
- net D7: track 41.1 -> 18.4 mm
- net CLK: track 47.2 -> 30.3 mm
- net Net-(INST_REG1-Pad5): track 125.6 -> 142.3 mm
- net D6: track 35.9 -> 20.9 mm
- net D4: track 18.3 -> 33.2 mm
- net D5: track 23.9 -> 29.6 mm
- net ~{ΣO}: track 54.7 -> 54.0 mm
- net H: track 30.7 -> 29.9 mm
- net C: track 36.1 -> 35.4 mm
- net Im: track 48.5 -> 47.8 mm
- net ~{II}: track 42.3 -> 41.6 mm
Other:
- board size 138.4 x 57.2 mm -> 139.7 x 58.5 mm

Commit message: add .readthedocs.yaml
Parts:
- U3: value AT28C16 -> 74HC161; footprint Package_DIP:DIP-24_W15.24mm_Socket -> Package_DIP:DIP-16_W7.62mm_Socket
- moved U3 4.58 mm to (171.4, 85.1)
Connections:
- INST_REG1 pad 12: Net-(INST_REG1-Pad12) -> Net-(U1-Pad4)
- INST_REG1 pad 15: Net-(INST_REG1-Pad15) -> Net-(U1-Pad3)
- INST_REG1 pad 16: Net-(INST_REG1-Pad16) -> Net-(U1-Pad2)
- INST_REG1 pad 19: Net-(INST_REG1-Pad19) -> Net-(U1-Pad1)
- INST_REG1 pad 2: Net-(INST_REG1-Pad2) -> Net-(U1-Pad8)
- INST_REG1 pad 5: Net-(INST_REG1-Pad5) -> Net-(U1-Pad7)
- INST_REG1 pad 6: Net-(INST_REG1-Pad6) -> Net-(U1-Pad6)
- INST_REG1 pad 9: Net-(INST_REG1-Pad9) -> Net-(U1-Pad5)
- U1 pad 1: Net-(INST_REG1-Pad19) -> Net-(U1-Pad1)
- U1 pad 19: GND -> Net-(U2-Pad19)
- U1 pad 2: Net-(INST_REG1-Pad16) -> Net-(U1-Pad2)
- U1 pad 22: GND -> Net-(U1-Pad22)
- U1 pad 23: GND -> Net-(U1-Pad23)
- U1 pad 3: Net-(INST_REG1-Pad15) -> Net-(U1-Pad3)
- U1 pad 4: Net-(INST_REG1-Pad12) -> Net-(U1-Pad4)
- U1 pad 5: Net-(INST_REG1-Pad9) -> Net-(U1-Pad5)
- U1 pad 6: Net-(INST_REG1-Pad6) -> Net-(U1-Pad6)
- U1 pad 7: Net-(INST_REG1-Pad5) -> Net-(U1-Pad7)
- U1 pad 8: Net-(INST_REG1-Pad2) -> Net-(U1-Pad8)
- U2 pad 1: Net-(INST_REG1-Pad19) -> Net-(U1-Pad1)
- U2 pad 19: GND -> Net-(U2-Pad19)
- U2 pad 2: Net-(INST_REG1-Pad16) -> Net-(U1-Pad2)
- U2 pad 22: GND -> Net-(U1-Pad22)
- U2 pad 23: GND -> Net-(U1-Pad23)
- U2 pad 3: Net-(INST_REG1-Pad15) -> Net-(U1-Pad3)
- U2 pad 4: Net-(INST_REG1-Pad12) -> Net-(U1-Pad4)
- U2 pad 5: Net-(INST_REG1-Pad9) -> Net-(U1-Pad5)
- U2 pad 6: Net-(INST_REG1-Pad6) -> Net-(U1-Pad6)
- U2 pad 7: Net-(INST_REG1-Pad5) -> Net-(U1-Pad7)
- U2 pad 8: Net-(INST_REG1-Pad2) -> Net-(U1-Pad8)
- U3 pad 1: Net-(INST_REG1-Pad19) -> Net-(U3-Pad1)
- U3 pad 11: unconnected-(U3-Pad11) -> Net-(U3-Pad1)
- U3 pad 12: GND -> Net-(U2-Pad19)
- U3 pad 13: unconnected-(U3-Pad13) -> Net-(U1-Pad22)
- U3 pad 14: unconnected-(U3-Pad14) -> Net-(U1-Pad23)
- U3 pad 16: unconnected-(U3-Pad16) -> +5V
- U3 pad 2: Net-(INST_REG1-Pad16) -> CLK
- U3 pad 3: Net-(INST_REG1-Pad15) -> unconnected-(U3-Pad3)
- U3 pad 4: Net-(INST_REG1-Pad12) -> unconnected-(U3-Pad4)
- U3 pad 5: Net-(INST_REG1-Pad9) -> unconnected-(U3-Pad5)
- U3 pad 6: Net-(INST_REG1-Pad6) -> unconnected-(U3-Pad6)
- U3 pad 7: Net-(INST_REG1-Pad5) -> +5V
- U3 pad 8: Net-(INST_REG1-Pad2) -> GND
Routing:
- net +5V: track 0.00 -> 152.3 mm
- net Net-(INST_REG1-Pad2): track 152.0 -> 0.00 mm
- net Net-(INST_REG1-Pad5): track 142.3 -> 0.00 mm
- net Net-(INST_REG1-Pad6): track 124.4 -> 0.00 mm
- net Net-(INST_REG1-Pad9): track 114.5 -> 0.00 mm
- net Net-(INST_REG1-Pad12): track 108.8 -> 0.00 mm
- net Net-(U1-Pad8): track 0.00 -> 95.9 mm
- net Net-(U1-Pad7): track 0.00 -> 90.2 mm
- net Net-(INST_REG1-Pad15): track 88.5 -> 0.00 mm
- net Net-(INST_REG1-Pad16): track 81.4 -> 0.00 mm
- net Net-(U1-Pad6): track 0.00 -> 76.3 mm
- net CLK: track 30.3 -> 100.7 mm
- net Net-(U1-Pad5): track 0.00 -> 70.3 mm
- net Net-(INST_REG1-Pad19): track 68.7 -> 0.00 mm
- net Net-(U1-Pad4): track 0.00 -> 68.6 mm
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- removed copper zone on In2.Cu, net +5V
Other:
- board size 139.7 x 58.5 mm -> 100.3 x 55.9 mm
- copper layers 4 -> 2
